File: Hardware/Placa_PCB/Power.kicad_sch (KiCad schematic)
At the start: 13 parts, among them J2 USB_C_Receptacle_PowerOnly_6P, J3 USB_C_Receptacle_USB2.0_16P, Q4 DMG2305UX-7

Commit message: Agregando MCU al esquematico
Parts:
- added C6: 1000uF, Capacitor_SMD:CP_Elec_6.3x5.4, symbol Device:C_Polarized
- added C7: 100nF, Capacitor_SMD:C_0805_2012Metric_Pad1.18x1.45mm_HandSolder, symbol Device:C
- added R12: 10k, Resistor_SMD:R_0805_2012Metric_Pad1.20x1.40mm_HandSolder, symbol Device:R
- added SW1: SW_SPST, symbol Switch:SW_SPST
- added U1: USBLC6-2SC6, Package_TO_SOT_SMD:SOT-23-6, symbol Power_Protection:USBLC6-2SC6
Connections:
- net +5V: now also C6.1
- net GNDD: now also C6.2, C7.2, R12.2, U1.2 (GND)
- net USB_D+: now also U1.1 (I/O1); no longer J3.A6 (D+), J3.B6 (D+)
- net USB_D-: now also U1.3 (I/O2); no longer J3.A7 (D-), J3.B7 (D-)
- net V_USB_POWER: now also SW1.1 (A); no longer Q4.3 (D)
- net V_USB_PROG: now also C7.1, U1.5 (VBUS)
- new net D+: J3.A6 (D+), J3.B6 (D+), U1.6 (I/O1)
- new net D-: J3.A7 (D-), J3.B7 (D-), U1.4 (I/O2)
- new net LED_USB: Q4.3 (D), R12.1, SW1.2 (B)
Other:
- note added: "PROTECCION EDS"
- moved on the sheet: C2, C3, C4, C5, D1, J2, J3, Q4, R10, R11, R7, R8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

Commit message: Esquematico Final
Parts:
- removed SW1: SW_SPST, symbol Switch:SW_SPST
- added SW1: POWER, Switch_3A:SW_100SP1T_12P7X6P86_EWI, symbol Switch:SW_Nidec_CAS-120A1
- C2, C4: footprint Capacitor_SMD:CP_Elec_6.3x5.4 -> Capacitor_SMD:CP_Elec_6.3x5.8
- C6: footprint Capacitor_SMD:CP_Elec_6.3x5.4 -> Capacitor_SMD:CP_Elec_10x10.5
- J2: footprint (none) -> Connector_USB:USB_C_Receptacle_GCT_USB4125-xx-x-0190_6P_TopMnt_Horizontal
- J3: footprint (none) -> Connector_USB:USB_C_Receptacle_HRO_TYPE-C-31-M-12
- renumbered U1 to U2
Connections:
- net LED_USB: now also SW1.1 (C)
- net V_USB_POWER: now also SW1.2 (B)
- no-connect marks 2 -> 3
Changed lines of the file:
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@@
 	)
 	(junction
-		(at 224.79 92.71)
-		(diameter 0)
-		(color 0 0 0 0)
-	)
-	(junction
 		(at 224.79 67.31)
 		(diameter 0)
@@
 		(at 143.51 86.36)
 	)
+	(no_connect
+		(at 238.76 50.8)
+	)
 	(wire
 		(pts
@@
 	(wire
 		(pts
-			(xy 245.11 53.34) (xy 246.38 53.34)
-		)
-		(stroke
-			(width 0)
-			(type default)
-		)
-	)
-	(wire
-		(pts
 			(xy 68.58 81.28) (xy 68.58 83.82)
 		)
@@
 	(wire
 		(pts
-			(xy 224.79 92.71) (xy 227.33 92.71)
-		)
-		(stroke
-			(width 0)
-			(type default)
-		)
-	)
-	(wire
-		(pts
 			(xy 246.38 48.26) (xy 246.38 53.34)
 		)
@@
 	(wire
 		(pts
-			(xy 232.41 53.34) (xy 234.95 53.34)
+			(xy 223.52 53.34) (xy 228.6 53.34)
 		)
 		(stroke
@@
 	(wire
 		(pts
-			(xy 224.79 92.71) (xy 224.79 93.98)
+			(xy 224.79 91.44) (xy 224.79 93.98)
 		)
 		(stroke
@@
 	(wire
 		(pts
+			(xy 238.76 55.88) (xy 240.03 55.88)
+		)
+		(stroke
+			(width 0)
+			(type default)
+		)
+	)
+	(wire
+		(pts
 			(xy 50.8 93.98) (xy 46.99 93.98)
 		)
@@
 	(wire
 		(pts
-			(xy 224.79 91.44) (xy 224.79 92.71)
-		)
-		(stroke
-			(width 0)
-			(type default)
-		)
-	)
-	(wire
-		(pts
 			(xy 68.58 93.98) (xy 73.66 93.98)
 		)
@@
 	(wire
 		(pts
+			(xy 240.03 53.34) (xy 246.38 53.34)
+		)
+		(stroke
+			(width 0)
+			(type default)
+		)
+	)
+	(wire
+		(pts
+			(xy 240.03 55.88) (xy 240.03 53.34)
+		)
+		(stroke
+			(width 0)
+			(type default)
+		)
+	)
+	(wire
+		(pts
 			(xy 182.88 49.53) (xy 187.96 49.53)
 		)
@@
 	)
 	(label "V_USB_POWER"
-		(at 232.41 53.34 180)
+		(at 223.52 53.34 180)
 		(effects
 			(font
@@
 		(on_board yes)
 		(dnp no)
-		(property "Reference" "U1"
+		(property "Reference" "U2"
 			(at 144.3989 119.38 0)
 			(effects
@@
 			(project "ScramblerBot"
 				(path "/ca162c4b-e7f6-494c-9ea1-0d86ef4a8e44/bb166e8a-7d54-4ae8-a0b2-867dec2483b7"
-					(reference "U1")
+					(reference "U2")
 					(unit 1)
 				)
@@
 			)
 		)
-		(property "Footprint" "Capacitor_SMD:CP_Elec_6.3x5.4"
+		(property "Footprint" "Capacitor_SMD:CP_Elec_6.3x5.8"
 			(at 172.4152 58.42 0)
 			(effects
@@
 	)
 	(symbol
+		(lib_id "Switch:SW_Nidec_CAS-120A1")
+		(at 233.68 53.34 0)
+		(unit 1)
+		(exclude_from_sim no)
+		(in_bom yes)
+		(on_board yes)
+		(dnp no)
+		(fields_autoplaced yes)
+		(property "Reference" "SW1"
+			(at 233.68 44.45 0)
+			(effects
+				(font
+					(size 1.27 1.27)
+				)
+			)
+		)
+		(property "Value" "POWER"
+			(at 233.68 46.99 0)
+			(effects
+				(font
+					(size 1.27 1.27)
+				)
+			)
+		)
+		(property "Footprint" "Switch_3A:SW_100SP1T_12P7X6P86_EWI"
+			(at 233.68 63.5 0)
+			(effects
+				(font
+					(size 1.27 1.27)
+				)
+				(hide yes)
+			)
+		)
+		(property "Datasheet" "https://www.nidec-components.com/e/catalog/switch/cas.pdf"
+			(at 233.68 60.96 0)
+			(effects
+				(font
+					(size 1.27 1.27)
+				)
+				(hide yes)
+			)
+		)
+		(property "Description" "Switch, single pole double throw"
+			(at 233.68 53.34 0)
+			(effects
+				(font
+					(size 1.27 1.27)
+				)
+				(hide yes)
+			)
+		)
+		(pin "2"
+		)
+		(pin "3"
+		)
+		(pin "1"
+		)
+		(instances
+			(project ""
+				(path "/ca162c4b-e7f6-494c-9ea1-0d86ef4a8e44/bb166e8a-7d54-4ae8-a0b2-867dec2483b7"
+					(reference "SW1")
+					(unit 1)
+				)
+			)
+		)
+	)
+	(symbol
 		(lib_id "Connector:USB_C_Receptacle_USB2.0_16P")
 		(at 128.27 71.12 0)
@@
 			)
 		)
-		(property "Footprint" ""
+		(property "Footprint" "Connector_USB:USB_C_Receptacle_HRO_TYPE-C-31-M-12"
 			(at 132.08 71.12 0)
 			(effects
@@
 	)
 	(symbol
-		(lib_id "power:PWR_FLAG")
-		(at 227.33 92.71 270)
-		(unit 1)
-		(exclude_from_sim no)
-		(in_bom yes)
-		(on_board yes)
-		(dnp no)
-		(fields_autoplaced yes)
-		(property "Reference" "#FLG02"
-			(at 229.235 92.71 0)
-			(effects
-				(font
-					(size 1.27 1.27)
-				)
-				(hide yes)
-			)
-		)
-		(property "Value" "PWR_FLAG"
-			(at 231.14 92.7099 90)
-			(effects
-				(font
-					(size 1.27 1.27)
-				)
-				(justify left)
-			)
-		)
-		(property "Footprint" ""
-			(at 227.33 92.71 0)
-			(effects
-				(font
-					(size 1.27 1.27)
-				)
-				(hide yes)
-			)
-		)
-		(property "Datasheet" "~"
-			(at 227.33 92.71 0)
-			(effects
-				(font
-					(size 1.27 1.27)
-				)
-				(hide yes)
-			)
-		)
-		(property "Description" "Special symbol for telling ERC where power comes from"
-			(at 227.33 92.71 0)
-			(effects
-				(font
-					(size 1.27 1.27)
-				)
-				(hide yes)
-			)
-		)
-		(pin "1"
-		)
-		(instances
-			(project "ScramblerBot"
-				(path "/ca162c4b-e7f6-494c-9ea1-0d86ef4a8e44/bb166e8a-7d54-4ae8-a0b2-867dec2483b7"
-					(reference "#FLG02")
-					(unit 1)
-				)
-			)
-		)
-	)
-	(symbol
 		(lib_id "Device:C")
 		(at 182.88 54.61 0)
@@
 			)
 		)
-		(property "Footprint" ""
+		(property "Footprint" "Connector_USB:USB_C_Receptacle_GCT_USB4125-xx-x-0190_6P_TopMnt_Horizontal"
 			(at 54.61 71.12 0)
 			(effects
@@
 			)
 		)
-		(property "Footprint" "Capacitor_SMD:CP_Elec_6.3x5.4"
+		(property "Footprint" "Capacitor_SMD:CP_Elec_6.3x5.8"
 			(at 77.1652 67.31 0)
 			(effects
@@
 			)
 		)
-		(property "Footprint" "Capacitor_SMD:CP_Elec_6.3x5.4"
+		(property "Footprint" "Capacitor_SMD:CP_Elec_10x10.5"
 			(at 247.3452 88.9 0)
 			(effects
@@
 					(unit 1)
 				)
-			)
-		)
-	)
-	(symbol
-		(lib_id "Switch:SW_SPST")
-		(at 240.03 53.34 0)
-		(unit 1)
-		(exclude_from_sim no)
-		(in_bom yes)
-		(on_board yes)
-		(dnp no)
-		(fields_autoplaced yes)
-		(property "Reference" "SW1"
-			(at 240.03 46.99 0)
-			(effects
-				(font
-					(size 1.27 1.27)
-				)
-			)
-		)
-		(property "Value" "SW_SPST"
-			(at 240.03 49.53 0)
-			(effects
-				(font
-					(size 1.27 1.27)
-				)
-			)
-		)
-		(property "Footprint" ""
-			(at 240.03 53.34 0)
-			(effects
-				(font
-					(size 1.27 1.27)
-				)
-				(hide yes)
-			)
-		)
-		(property "Datasheet" "~"
-			(at 240.03 53.34 0)
-			(effects
-				(font
-					(size 1.27 1.27)
-				)
-				(hide yes)
-			)
-		)
-		(property "Description" "Single Pole Single Throw (SPST) switch"
-			(at 240.03 53.34 0)
-			(effects
-				(font
-					(size 1.27 1.27)
-				)
-				(hide yes)
-			)
-		)
-		(pin "2"
-		)
-		(pin "1"
-		)
-		(instances
-			(project "ScramblerBot"
-				(path "/ca162c4b-e7f6-494c-9ea1-0d86ef4a8e44/bb166e8a-7d54-4ae8-a0b2-867dec2483b7"
-					(reference "SW1")
-					(unit 1)
-				)
