File: Hardware/Placa_PCB/Camara.kicad_sch (KiCad schematic)
At the start: 3 parts, among them J8 Conn_01x08_Pin

Commit message: Agregando MCU al esquematico
Parts:
- renumbered C10 to C14, C12 to C15
Changed lines of the file:
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@@
 	)
 	(hierarchical_label "MISO"
-		(shape input)
+		(shape output)
 		(at 127 92.71 90)
 		(effects
@@
 		(on_board yes)
 		(dnp no)
-		(property "Reference" "C12"
+		(property "Reference" "C15"
 			(at 160.02 100.076 90)
 			(effects
@@
 			(project ""
 				(path "/ca162c4b-e7f6-494c-9ea1-0d86ef4a8e44/978087f4-bf8d-48ff-9a7b-a9e2b1e602ee"
-					(reference "C12")
+					(reference "C15")
 					(unit 1)
 				)
@@
 		(dnp no)
 		(fields_autoplaced yes)
-		(property "Reference" "C10"
+		(property "Reference" "C14"
 			(at 160.909 82.55 90)
 			(effects
@@
 			(project ""
 				(path "/ca162c4b-e7f6-494c-9ea1-0d86ef4a8e44/978087f4-bf8d-48ff-9a7b-a9e2b1e602ee"
-					(reference "C10")
-					(unit 1)
-				)
+					(reference "C14")
+					(unit 1)
+				)

Commit message: Esquematico Final
Parts:
- C14: footprint Capacitor_SMD:CP_Elec_6.3x5.2 -> Capacitor_SMD:CP_Elec_6.3x5.8
- J8: footprint (none) -> Connector_PinHeader_2.54mm:PinHeader_1x08_P2.54mm_Vertical
Changed lines of the file:
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@@
 			)
 		)
-		(property "Footprint" ""
+		(property "Footprint" "Connector_PinHeader_2.54mm:PinHeader_1x08_P2.54mm_Vertical"
 			(at 129.54 100.33 0)
 			(effects
@@
 			)
 		)
-		(property "Footprint" "Capacitor_SMD:CP_Elec_6.3x5.2"
+		(property "Footprint" "Capacitor_SMD:CP_Elec_6.3x5.8"
 			(at 156.21 91.1352 0)
 			(effects

Commit message: Actualizacion de PCB con rellenos ordenados, solo falta colocar las vias
Parts:
- removed C14: 100uF, Capacitor_SMD:CP_Elec_6.3x5.8, symbol Device:C_Polarized
- added C14: 10uF, Capacitor_SMD:C_0805_2012Metric_Pad1.18x1.45mm_HandSolder, symbol Device:C
Connections:
- net +5V: now also C14.2
- net GNDD: now also C14.1
Changed lines of the file:
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@@
+	)
+	(symbol
+		(lib_id "Device:C")
+		(at 160.02 90.17 90)
+		(unit 1)
+		(exclude_from_sim no)
+		(in_bom yes)
+		(on_board yes)
+		(dnp no)
+		(fields_autoplaced yes)
+		(property "Reference" "C14"
+			(at 160.02 82.55 90)
+			(effects
+				(font
+					(size 1.27 1.27)
+				)
+			)
+		)
+		(property "Value" "10uF"
+			(at 160.02 85.09 90)
+			(effects
+				(font
+					(size 1.27 1.27)
+				)
+			)
+		)
+		(property "Footprint" "Capacitor_SMD:C_0805_2012Metric_Pad1.18x1.45mm_HandSolder"
+			(at 163.83 89.2048 0)
+			(effects
+				(font
+					(size 1.27 1.27)
+				)
+				(hide yes)
+			)
+		)
+		(property "Datasheet" "~"
+			(at 160.02 90.17 0)
+			(effects
+				(font
+					(size 1.27 1.27)
+				)
+				(hide yes)
+			)
+		)
+		(property "Description" "Unpolarized capacitor"
+			(at 160.02 90.17 0)
+			(effects
+				(font
+					(size 1.27 1.27)
+				)
+				(hide yes)
+			)
+		)
+		(pin "1"
+		)
+		(pin "2"
+		)
+		(instances
+			(project ""
+				(path "/ca162c4b-e7f6-494c-9ea1-0d86ef4a8e44/978087f4-bf8d-48ff-9a7b-a9e2b1e602ee"
+					(reference "C14")
+					(unit 1)
+				)
+			)
+		)
 	)
 	(symbol
@@
 					(unit 1)
 				)
-			)
-		)
-	)
-	(symbol
-		(lib_id "Device:C_Polarized")
-		(at 160.02 90.17 270)
-		(unit 1)
-		(exclude_from_sim no)
-		(in_bom yes)
-		(on_board yes)
-		(dnp no)
-		(fields_autoplaced yes)
-		(property "Reference" "C14"
-			(at 160.909 82.55 90)
-			(effects
-				(font
-					(size 1.27 1.27)
-				)
-			)
-		)
-		(property "Value" "100uF"
-			(at 160.909 85.09 90)
-			(effects
-				(font
-					(size 1.27 1.27)
-				)
-			)
-		)
-		(property "Footprint" "Capacitor_SMD:CP_Elec_6.3x5.8"
-			(at 156.21 91.1352 0)
-			(effects
-				(font
-					(size 1.27 1.27)
-				)
-				(hide yes)
-			)
-		)
-		(property "Datasheet" "~"
-			(at 160.02 90.17 0)
-			(effects
-				(font
-					(size 1.27 1.27)
-				)
-				(hide yes)
-			)
-		)
-		(property "Description" "Polarized capacitor"
-			(at 160.02 90.17 0)
-			(effects
-				(font
-					(size 1.27 1.27)
-				)
-				(hide yes)
-			)
-		)
-		(pin "1"
-		)
-		(pin "2"
-		)
-		(instances
-			(project ""
-				(path "/ca162c4b-e7f6-494c-9ea1-0d86ef4a8e44/978087f4-bf8d-48ff-9a7b-a9e2b1e602ee"
-					(reference "C14")
-					(unit 1)
-				)
